File: DZAS7265X-PCB/AS7265X-Sensor.sch (KiCad schematic (older format))
At the start: 3 parts

Commit message: Finalizacao esquema
Finalizacao projeto esquematico
Parts:
- added C10, C12, C14: C0805C105K4RACTU, Capacitor_SMD:C_0805_2012Metric, symbol Device:C
- added C11, C13, C15: 0805B104J500CT, Capacitor_SMD:C_0805_2012Metric, symbol Device:C
- added D3: L1SP-PNK1002800000, Resistor_SMD:R_1206_3216Metric, symbol Device:LED
- added D4, D6, D8: LED, symbol Device:LED
- added D5: L1SP-FRD0002800000, Resistor_SMD:R_1206_3216Metric, symbol Device:LED
- added D7: SIR67-21C/TR8, Resistor_SMD:R_1206_3216Metric, symbol Device:LED
- added R10, R11, R12, R8: CRCW080510K0JNEA, Resistor_SMD:R_0805_2012Metric, symbol Device:R
- added R13: CRCW080533R0JNEA, Resistor_SMD:R_0805_2012Metric, symbol Device:R
- added R14, R15: CRCW0805100RJNEAC, Resistor_SMD:R_0805_2012Metric, symbol Device:R
- added R9: CRCW08050000Z0EA, Resistor_SMD:R_0805_2012Metric, symbol Device:R
- U4: renamed from U?; Desc (none) -> SMART VIS-NIR SPECTRAL SENSOR; PN_DIGIKEY (none) -> AS72651-BLGTTR-ND; PRICE_DIGIKEY (none) -> 7.22
- U5: renamed from U?; Desc (none) -> SMART VIS-NIR SPECTRAL SENSOR; PN_DIGIKEY (none) -> AS72652-BLGTTR-ND; PRICE_DIGIKEY (none) -> 7.22
- U6: renamed from U?; Desc (none) -> SMART VIS-NIR SPECTRAL SENSOR; PN_DIGIKEY (none) -> AS72653-BLGTTR-ND; PRICE_DIGIKEY (none) -> 7.22
Connections:
- net +3V3: now also C10.1, C11.1, C12.1, C13.1, C14.1, C15.1, D4.2 (A), D6.2 (A), D8.2 (A), R10.1, R11.1, R12.1, R8.1
- net GND: now also C10.2, C11.2, C12.2, C13.2, C14.2, C15.2, R9.2
- net SLV1_RESN: now reaches U4.1 (SLV1_RESN)
- net SLV1_RESN: now also U5.2 (RESN), R11.2
- net INT: now reaches U4.13 (INT)
- net at U4.15 (LED_DRV): now also D3.1 (K)
- net at U4.18 (LED_IND): now also D4.1 (K)
- net RESN: now reaches U4.2 (RESN)
- net RESN: now also R10.2
- net SLV2_RESN: now reaches U4.20 (SLV2_RESN)
- net SLV2_RESN: now also U6.2 (RESN), R12.2
- net at U4.8 (I2C_ENB): now also R8.2, R9.1
- net at U5.15 (LED_DRV): now also D5.1 (K)
- net at U5.18 (LED_IND): now also D6.1 (K)
- net at U6.15 (LED_DRV): now also D7.1 (K)
- net at U6.18 (LED_IND): now also D8.1 (K)
- new net: D3.2 (A), R13.2
- new net: D5.2 (A), R14.2
- new net: D7.2 (A), R15.2
- new net +5V: R13.1, R14.1, R15.1
Other:
- moved on the sheet: U4, U6

Commit message: Atualização para lista de compra
Parts:
- C10, C12, C14: PN_DIGIKEY 399-1284-2-ND -> 399-1284-1-ND
- D3: PN_DIGIKEY 1416-2062-2-ND -> 1416-2062-1-ND
- D4, D6, D8: value LED -> LG R971-KN-1; footprint (none) -> LED_SMD:LED_0805_2012Metric; Desc (none) -> LED GRN DIF 2.2V 20MA 0805; PN_DIGIKEY (none) -> 475-1410-1-ND; PRICE_DIGIKEY (none) -> 0.26
- D5: PN_DIGIKEY 1416-2055-2-ND -> 1416-2055-1-ND
- D7: PN_DIGIKEY 1080-1427-2-ND -> 1080-1427-1-ND
- R10, R11, R12, R8: PN_DIGIKEY 541-10KATR-ND -> 541-10KACT-ND
- U4: symbol AS72651:AS72651-BLGT -> DZAS7265X-PCB-rescue:AS72651-BLGT-AS72651; MANUFACTURER AMS -> (none); PARTREV 1-04 -> (none); STANDARD IPC-7351B -> (none)
- U5: symbol AS72652:AS72652-BLGT -> DZAS7265X-PCB-rescue:AS72652-BLGT-AS72652; MANUFACTURER AMS -> (none); PARTREV 1-04 -> (none); STANDARD IPC-7351B -> (none)
- U6: symbol AS72653:AS72653-BLGT -> DZAS7265X-PCB-rescue:AS72653-BLGT-AS72653; MANUFACTURER AMS -> (none); PARTREV 1-04 -> (none); STANDARD IPC-7351B -> (none)
Changed lines of the file:
@@
 $EndDescr
 $Comp
-L AS72651:AS72651-BLGT U?
+L DZAS7265X-PCB-rescue:AS72651-BLGT-AS72651 U?
 U 1 1 6155508F
 P 2300 2150
@@
 F 2 "PQFN65P470X450X270-20N" H 2300 1950 50  0001 L BNN
 F 3 "https://ams.com/documents/20143/36005/AS7265x_DS000612_1-00.pdf/08051c8a-a7f6-6231-7993-2d3fe0bf38b8" H 2300 2150 50  0001 L BNN
-F 4 "IPC-7351B" H 2300 1850 50  0001 L BNN "STANDARD"
-F 5 "AMS" H 2300 2050 50  0001 L BNN "MANUFACTURER"
-F 6 "1-04" H 2300 1750 50  0001 L BNN "PARTREV"
-F 7 "SMART VIS-NIR SPECTRAL SENSOR" H 2300 2150 50  0001 C CNN "Desc"
-F 8 "AS72651-BLGTTR-ND" H 2300 2150 50  0001 C CNN "PN_DIGIKEY"
-F 9 "7.22" H 2300 2150 50  0001 C CNN "PRICE_DIGIKEY"
+F 4 "SMART VIS-NIR SPECTRAL SENSOR" H 2300 2150 50  0001 C CNN "Desc"
+F 5 "AS72651-BLGTTR-ND" H 2300 2150 50  0001 C CNN "PN_DIGIKEY"
+F 6 "7.22" H 2300 2150 50  0001 C CNN "PRICE_DIGIKEY"
 	1    2300 2150
 	1    0    0    -1
 $EndComp
 $Comp
-L AS72652:AS72652-BLGT U?
+L DZAS7265X-PCB-rescue:AS72652-BLGT-AS72652 U?
 U 1 1 61555098
 P 5600 2175
@@
 F 2 "PQFN65P470X450X270-20N" H 5600 1975 50  0001 L BNN
 F 3 "https://ams.com/documents/20143/36005/AS7265x_DS000612_1-00.pdf/08051c8a-a7f6-6231-7993-2d3fe0bf38b8" H 5600 2175 50  0001 L BNN
-F 4 "IPC-7351B" H 5600 1875 50  0001 L BNN "STANDARD"
-F 5 "AMS" H 5600 2075 50  0001 L BNN "MANUFACTURER"
-F 6 "1-04" H 5600 1775 50  0001 L BNN "PARTREV"
-F 7 "SMART VIS-NIR SPECTRAL SENSOR" H 5600 2175 50  0001 C CNN "Desc"
-F 8 "AS72652-BLGTTR-ND" H 5600 2175 50  0001 C CNN "PN_DIGIKEY"
-F 9 "7.22" H 5600 2175 50  0001 C CNN "PRICE_DIGIKEY"
+F 4 "SMART VIS-NIR SPECTRAL SENSOR" H 5600 2175 50  0001 C CNN "Desc"
+F 5 "AS72652-BLGTTR-ND" H 5600 2175 50  0001 C CNN "PN_DIGIKEY"
+F 6 "7.22" H 5600 2175 50  0001 C CNN "PRICE_DIGIKEY"
 	1    5600 2175
 	1    0    0    -1
 $EndComp
 $Comp
-L AS72653:AS72653-BLGT U?
+L DZAS7265X-PCB-rescue:AS72653-BLGT-AS72653 U?
 U 1 1 615550A1
 P 9100 2225
@@
 F 2 "PQFN65P470X450X270-20N" H 9100 2025 50  0001 L BNN
 F 3 "https://ams.com/documents/20143/36005/AS7265x_DS000612_1-00.pdf/08051c8a-a7f6-6231-7993-2d3fe0bf38b8" H 9100 2225 50  0001 L BNN
-F 4 "IPC-7351B" H 9100 1925 50  0001 L BNN "STANDARD"
-F 5 "AMS" H 9100 2125 50  0001 L BNN "MANUFACTURER"
-F 6 "1-04" H 9100 1825 50  0001 L BNN "PARTREV"
-F 7 "SMART VIS-NIR SPECTRAL SENSOR" H 9100 2225 50  0001 C CNN "Desc"
-F 8 "AS72653-BLGTTR-ND" H 9100 2225 50  0001 C CNN "PN_DIGIKEY"
-F 9 "7.22" H 9100 2225 50  0001 C CNN "PRICE_DIGIKEY"
+F 4 "SMART VIS-NIR SPECTRAL SENSOR" H 9100 2225 50  0001 C CNN "Desc"
+F 5 "AS72653-BLGTTR-ND" H 9100 2225 50  0001 C CNN "PN_DIGIKEY"
+F 6 "7.22" H 9100 2225 50  0001 C CNN "PRICE_DIGIKEY"
 	1    9100 2225
 	1    0    0    -1
@@
 F 4 "CAP CER 1UF 10% 10V X7R 0805" H 2425 3925 50  0001 C CNN "Desc"
 F 5 "1uF" H 1850 4075 50  0000 C CNN "Comment"
-F 6 "399-1284-2-ND" H 1750 4000 50  0001 C CNN "PN_DIGIKEY"
+F 6 "399-1284-1-ND" H 1750 4000 50  0001 C CNN "PN_DIGIKEY"
 F 7 "0.14" H 1750 4000 50  0001 C CNN "PRICE_DIGIKEY"
 	1    1750 4000
@@
 F 4 "CAP CER 1UF 10% 10V X7R 0805" H 5725 3975 50  0001 C CNN "Desc"
 F 5 "1uF" H 5150 4125 50  0000 C CNN "Comment"
-F 6 "399-1284-2-ND" H 5050 4050 50  0001 C CNN "PN_DIGIKEY"
+F 6 "399-1284-1-ND" H 5050 4050 50  0001 C CNN "PN_DIGIKEY"
 F 7 "0.14" H 5050 4050 50  0001 C CNN "PRICE_DIGIKEY"
 	1    5050 4050
@@
 F 4 "CAP CER 1UF 10% 10V X7R 0805" H 9225 4000 50  0001 C CNN "Desc"
 F 5 "1uF" H 8650 4150 50  0000 C CNN "Comment"
-F 6 "399-1284-2-ND" H 8550 4075 50  0001 C CNN "PN_DIGIKEY"
+F 6 "399-1284-1-ND" H 8550 4075 50  0001 C CNN "PN_DIGIKEY"
 F 7 "0.14" H 8550 4075 50  0001 C CNN "PRICE_DIGIKEY"
 	1    8550 4075
@@
 F 3 "https://www.lumileds.com/wp-content/uploads/files/DS237-luxeon-sunplus-2835-line-datasheet.pdf" H 3625 1725 50  0001 C CNN
 F 4 "LUXEON SUNPLUS 2835 WHITE" H 3625 1725 50  0001 C CNN "Desc"
-F 5 "1416-2062-2-ND" H 3625 1725 50  0001 C CNN "PN_DIGIKEY"
+F 5 "1416-2062-1-ND" H 3625 1725 50  0001 C CNN "PN_DIGIKEY"
 F 6 "0.63" H 3625 1725 50  0001 C CNN "PRICE_DIGIKEY"
 	1    3625 1725
@@
 AR Path="/61548E0F/60854701" Ref="D4"  Part="1"
 F 0 "D4" H 3825 2325 50  0000 R CNN
-F 1 "LED" H 3875 2250 50  0000 R CNN
-F 2 "" H 3825 2150 50  0001 C CNN
-F 3 "~" H 3825 2150 50  0001 C CNN
+F 1 "LG R971-KN-1" H 4050 2000 50  0000 R CNN
+F 2 "LED_SMD:LED_0805_2012Metric" H 3825 2150 50  0001 C CNN
+F 3 "https://dammedia.osram.info/media/resource/hires/osram-dam-14795755/LG%20R971_EN.pdf" H 3825 2150 50  0001 C CNN
+F 4 "LED GRN DIF 2.2V 20MA 0805" H 3825 2150 50  0001 C CNN "Desc"
+F 5 "475-1410-1-ND" H 3825 2150 50  0001 C CNN "PN_DIGIKEY"
+F 6 "0.26" H 3825 2150 50  0001 C CNN "PRICE_DIGIKEY"
 	1    3825 2150
 	1    0    0    -1
@@
 F 3 "https://www.lumileds.com/wp-content/uploads/files/DS237-luxeon-sunplus-2835-line-datasheet.pdf" H 6925 1750 50  0001 C CNN
 F 4 "LUXEON SUNPLUS 2835 FAR RED" H 6925 1750 50  0001 C CNN "Desc"
-F 5 "1416-2055-2-ND" H 6925 1750 50  0001 C CNN "PN_DIGIKEY"
+F 5 "1416-2055-1-ND" H 6925 1750 50  0001 C CNN "PN_DIGIKEY"
 F 6 "0.69" H 6925 1750 50  0001 C CNN "PRICE_DIGIKEY"
 	1    6925 1750
@@
 AR Path="/61548E0F/6085ED8D" Ref="D6"  Part="1"
 F 0 "D6" H 7125 2350 50  0000 R CNN
-F 1 "LED" H 7175 2275 50  0000 R CNN
-F 2 "" H 7125 2175 50  0001 C CNN
-F 3 "~" H 7125 2175 50  0001 C CNN
+F 1 "LG R971-KN-1" H 7350 2000 50  0000 R CNN
+F 2 "LED_SMD:LED_0805_2012Metric" H 7125 2175 50  0001 C CNN
+F 3 "https://dammedia.osram.info/media/resource/hires/osram-dam-14795755/LG%20R971_EN.pdf" H 7125 2175 50  0001 C CNN
+F 4 "LED GRN DIF 2.2V 20MA 0805" H 7125 2175 50  0001 C CNN "Desc"
+F 5 "475-1410-1-ND" H 7125 2175 50  0001 C CNN "PN_DIGIKEY"
+F 6 "0.26" H 7125 2175 50  0001 C CNN "PRICE_DIGIKEY"
 	1    7125 2175
 	1    0    0    -1
@@
 F 3 "https://www.everlight.com/file/ProductFile/201407052129409395.pdf" H 10425 1800 50  0001 C CNN
 F 4 "EMITTER IR 875NM 65MA SMD" H 10425 1800 50  0001 C CNN "Desc"
-F 5 "1080-1427-2-ND" H 10425 1800 50  0001 C CNN "PN_DIGIKEY"
+F 5 "1080-1427-1-ND" H 10425 1800 50  0001 C CNN "PN_DIGIKEY"
 F 6 "0.64" H 10425 1800 50  0001 C CNN "PRICE_DIGIKEY"
 	1    10425 1800
@@
 AR Path="/61548E0F/608634FE" Ref="D8"  Part="1"
 F 0 "D8" H 10625 2400 50  0000 R CNN
-F 1 "LED" H 10675 2325 50  0000 R CNN
-F 2 "" H 10625 2225 50  0001 C CNN
-F 3 "~" H 10625 2225 50  0001 C CNN
+F 1 "LG R971-KN-1" H 10850 2050 50  0000 R CNN
+F 2 "LED_SMD:LED_0805_2012Metric" H 10625 2225 50  0001 C CNN
+F 3 "https://dammedia.osram.info/media/resource/hires/osram-dam-14795755/LG%20R971_EN.pdf" H 10625 2225 50  0001 C CNN
+F 4 "LED GRN DIF 2.2V 20MA 0805" H 10625 2225 50  0001 C CNN "Desc"
+F 5 "475-1410-1-ND" H 10625 2225 50  0001 C CNN "PN_DIGIKEY"
+F 6 "0.26" H 10625 2225 50  0001 C CNN "PRICE_DIGIKEY"
 	1    10625 2225
 	1    0    0    -1
@@
 F 4 "RES SMD 10K OHM 5% 1/8W 0805" H 3525 3850 50  0001 C CNN "Desc"
 F 5 "10k" H 2850 4075 50  0000 C CNN "Comment"
-F 6 "541-10KATR-ND" H 2775 3925 50  0001 C CNN "PN_DIGIKEY"
+F 6 "541-10KACT-ND" H 2775 3925 50  0001 C CNN "PN_DIGIKEY"
 F 7 "0.10" H 2775 3925 50  0001 C CNN "PRICE_DIGIKEY"
 	1    2775 3925
@@
 F 4 "RES SMD 10K OHM 5% 1/8W 0805" H 3800 3850 50  0001 C CNN "Desc"
 F 5 "10k" H 3125 4075 50  0000 C CNN "Comment"
-F 6 "541-10KATR-ND" H 3050 3925 50  0001 C CNN "PN_DIGIKEY"
+F 6 "541-10KACT-ND" H 3050 3925 50  0001 C CNN "PN_DIGIKEY"
 F 7 "0.10" H 3050 3925 50  0001 C CNN "PRICE_DIGIKEY"
 	1    3050 3925
@@
 F 4 "RES SMD 10K OHM 5% 1/8W 0805" H 4075 3850 50  0001 C CNN "Desc"
 F 5 "10k" H 3400 4075 50  0000 C CNN "Comment"
-F 6 "541-10KATR-ND" H 3325 3925 50  0001 C CNN "PN_DIGIKEY"
+F 6 "541-10KACT-ND" H 3325 3925 50  0001 C CNN "PN_DIGIKEY"
 F 7 "0.10" H 3325 3925 50  0001 C CNN "PRICE_DIGIKEY"
 	1    3325 3925
@@
 F 4 "RES SMD 10K OHM 5% 1/8W 0805" H 1400 1525 50  0001 C CNN "Desc"
 F 5 "10k" H 725 1750 50  0000 C CNN "Comment"
-F 6 "541-10KATR-ND" H 650 1600 50  0001 C CNN "PN_DIGIKEY"
+F 6 "541-10KACT-ND" H 650 1600 50  0001 C CNN "PN_DIGIKEY"
 F 7 "0.10" H 650 1600 50  0001 C CNN "PRICE_DIGIKEY"
 	1    650  1600
