File: DZAS7265X-PCB/FTDI-USB-Converter.sch (KiCad schematic (older format))
At the start: 26 parts

Commit message: Finalizacao esquema
Finalizacao projeto esquematico
Parts:
- removed D? (x6): CG0603MLU-12E, Diode_SMD:D_0603_1608Metric, symbol Device:D_TVS
- removed J?: USB_OTG, symbol Connector:USB_OTG
- added J1: USB3100-30-A, GCT_USB3100-XX-X_REVB, symbol USB3100-XX-X_REVB:USB3100-XX-X_REVB
- C1, C3: renamed from C?; value 0603B103J250C -> 0805B103K250CT; footprint Capacitor_SMD:C_0603_1608Metric -> Capacitor_SMD:C_0805_2012Metric; Desc CAP CER 10000PF 5% 25V X7R 0603 -> CAP CER 10000PF 10% 25V X7R 0805; PN_DIGIKEY (none) -> 1292-1561-2-ND; PRICE_DIGIKEY (none) -> 0.11
- C2, C6: renamed from C?; value 0603B104J250CT -> 0805B104J500CT; footprint Capacitor_SMD:C_0603_1608Metric -> Capacitor_SMD:C_0805_2012Metric; Desc CAP CER 0.1UF 5% 25V X7R 0603 -> CAP CER 0.1UF 5% 25V X7R 0805; PN_DIGIKEY (none) -> 1292-1564-1-ND; PRICE_DIGIKEY (none) -> 0.18
- C4, C5: renamed from C?; value 0603ZD106KAT2A -> C0805C106K8PACTU; footprint Capacitor_SMD:C_0603_1608Metric -> Capacitor_SMD:C_0805_2012Metric; Desc CAP CER 10UF 10% 10V X5R 0603 -> CAP CER 10UF 10% 10V X5R 0805; PN_DIGIKEY (none) -> 399-4925-2-ND; PRICE_DIGIKEY (none) -> 0.15
- C7: renamed from C?; value 0603ZD475KAT2A -> C0805C475K4PACTU; footprint Capacitor_SMD:C_0603_1608Metric -> Capacitor_SMD:C_0805_2012Metric; Desc CAP CER 4.7UF 10% 10V X5R 0603 -> CAP CER 4.7UF 10% 10V X7R 0805; PN_DIGIKEY (none) -> 399-8101-2-ND; PRICE_DIGIKEY (none) -> 0.28
- FB1: renamed from FB?; value CZP2BFTTE800P -> BLM21PG221SZ1D; footprint Inductor_SMD:L_1206_3216Metric -> Capacitor_SMD:C_0805_2012Metric; Desc Ferrite Beads 1206 80R 25% -> FERRITE BEAD 220 OHM 2A 0805; PN_DIGIKEY (none) -> 490-16661-2-ND; PRICE_DIGIKEY (none) -> 0.12
- R1, R2, R3, R4, R7: renamed from R?; value CRCW060310K0JNEA -> CRCW080510K0JNEA; footprint Resistor_SMD:R_0603_1608Metric -> Resistor_SMD:R_0805_2012Metric; Desc RES SMD 10K OHM 5% 1/10W 0603 -> RES SMD 10K OHM 5% 1/8W 0805; PN_DIGIKEY (none) -> 541-10KATR-ND; PRICE_DIGIKEY (none) -> 0.10
- R5, R6: renamed from R?; value CRCW0603270RJNEA -> CRCW0805270RJNEA; footprint Resistor_SMD:R_0603_1608Metric -> Resistor_SMD:R_0805_2012Metric; Desc RES SMD 270 OHM 5% 1/10W 0603 -> RES SMD 270 OHM 5% 1/8W 0805; PN_DIGIKEY (none) -> 541-270ATR-ND; PRICE_DIGIKEY (none) -> 0.10
- U1: renamed from U?; Desc (none) -> IC USB FS SERIAL UART 32-QFN; PN_DIGIKEY (none) -> 768-1008-2-ND; PRICE_DIGIKEY (none) -> 4.60
- U2: renamed from U?; Desc (none) -> AUTOMOTIVE LDO 1-A, LOW-IQ, HIGH-PSR; PN_DIGIKEY (none) -> 296-TPS74633PQWDRBRQ1TR-ND; PRICE_DIGIKEY (none) -> 1.32
- gave numbers to parts that had none: 2
Connections:
- net D+: now also J1.2 (D-)
- net D-: now also J1.3 (D+)
- net GND: now also J1.4 (ID), J1.5 (GND), J1.6 (SHIELD), J1.7 (SHIELD), J1.8 (SHIELD), J1.9 (SHIELD)
- net at FB1.2: now also J1.1 (VBUS)
Other:
- moved on the sheet: C1, C6, C7, D1, D2, FB1, R1, R2, R3, R4, R5, R6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

Commit message: Atualização para lista de compra
Parts:
- C1, C3: PN_DIGIKEY 1292-1561-2-ND -> 1292-1561-1-ND
- C4, C5: PN_DIGIKEY 399-4925-2-ND -> 399-4925-1-ND
- C7: PN_DIGIKEY 399-8101-2-ND -> 399-8101-1-ND
- D1, D2: value LED -> LG R971-KN-1; footprint (none) -> LED_SMD:LED_0805_2012Metric; Desc (none) -> LED GRN DIF 2.2V 20MA 0805; PN_DIGIKEY (none) -> 475-1410-1-ND; PRICE_DIGIKEY (none) -> 0.26
- FB1: PN_DIGIKEY 490-16661-2-ND -> 490-16661-1-ND
- J1: MANUFACTURER GCT -> (none)
- R1, R2, R3, R4, R7: PN_DIGIKEY 541-10KATR-ND -> 541-10KACT-ND
- U1: A_MAX 0.9 -> (none); B_MAX 0.3 -> (none); B_MIN 0.2 -> (none); B_NOM 0.25 -> (none); D2_NOM 3.4 -> (none); D_MAX 5.0 -> (none); D_MIN 5.0 -> (none); D_NOM 5.0 -> (none); E2_NOM 3.4 -> (none); ENOM 0.5 -> (none); E_MAX 5.0 -> (none); E_MIN 5.0 -> (none); E_NOM 5.0 -> (none); L_MAX 0.45 -> (none); L_MIN 0.35 -> (none); L_NOM 0.4 -> (none); MANUFACTURER FTDI -> (none); MAXIMUM_PACKAGE_HEIGHT 0.9mm -> (none); PARTREV 2.15 -> (none); PIN_COUNT_D 8.0 -> (none); PIN_COUNT_E 8.0 -> (none); PN_DIGIKEY 768-1008-2-ND -> 768-1008-1-ND; SNAPEDA_PACKAGE_ID 71296 -> (none); STANDARD IPC 7351B -> (none)
- U2: symbol Regulator_Linear:TPS74633PQWDRBRQ1 -> DZAS7265X-PCB-rescue:TPS74633PQWDRBRQ1-Regulator_Linear
