File: DZAS7265X-PCB/SPI-Flash-Memory.sch (KiCad schematic (older format))
At the start: 8 parts

Commit message: Finalizacao esquema
Finalizacao projeto esquematico
Parts:
- C8: renamed from C?; value C0603C105K8PACTU -> C0805C105K4RACTU; footprint Capacitor_SMD:C_0603_1608Metric -> Capacitor_SMD:C_0805_2012Metric; Desc CAP CER 1UF 10% 10V X5R 0603 -> CAP CER 1UF 10% 10V X7R 0805; PN_DIGIKEY (none) -> 399-1284-2-ND; PRICE_DIGIKEY (none) -> 0.14
- C9: renamed from C?; value 0603B104J250CT -> 0805B104J500CT; footprint Capacitor_SMD:C_0603_1608Metric -> Capacitor_SMD:C_0805_2012Metric; Desc CAP CER 0.1UF 5% 25V X7R 0603 -> CAP CER 0.1UF 5% 25V X7R 0805; PN_DIGIKEY (none) -> 1292-1564-1-ND; PRICE_DIGIKEY (none) -> 0.18
- FB2: renamed from FB?; value 742792653 -> BLM21BD601SH1D; footprint Inductor_SMD:L_1206_3216Metric -> Capacitor_SMD:C_0805_2012Metric; Desc Ferrite Beads 0603 600R 0.3A -> FERRITE BEAD 600 OHM 300mA 0805; PN_DIGIKEY (none) -> 490-11047-2-ND; PRICE_DIGIKEY (none) -> 0.18
- J2: renamed from J?; value Conn_01x07_Female -> 0022032071; Desc (none) -> CONN HEADER VERT 7 POS 2.54MM; PN_DIGIKEY (none) -> WM4005-ND; PRICE_DIGIKEY (none) -> 0.72
- J3: renamed from J?; Desc (none) -> CABLE ADAPTER 6 POS
- J4: renamed from J?; Desc (none) -> CONN FPC BOTTOM 8POS 0.50MM R/A; PN_DIGIKEY (none) -> A100281TR-ND; PRICE_DIGIKEY (none) -> 0.46
- Q1: renamed from Q?; Desc (none) -> TRANS PREBIAS NPN 200MW UMT3; PN_DIGIKEY (none) -> DTC113ZUAT106TR-ND; PRICE_DIGIKEY (none) -> 0.20
- U3: renamed from U?; Desc (none) -> IC FLASH 4MBIT SPI/QUAD 8SOIC; PN_DIGIKEY (none) -> 1265-AT25SF041B-SHD-B-ND; PRICE_DIGIKEY (none) -> 0.36
Other:
- moved on the sheet: J2, J4

Commit message: Atualização para lista de compra
Parts:
- C8: PN_DIGIKEY 399-1284-2-ND -> 399-1284-1-ND
- FB2: PN_DIGIKEY 490-11047-2-ND -> 490-11047-1-ND
- J3: MANUFACTURER Tag-Connect -> (none); PARTREV MS -> (none); STANDARD Manufacturer recommendation -> (none)
- J4: MANUFACTURER TE Connectivity -> (none); MAXIMUM_PACKAGE_HEIGHT 2.05mm -> (none); PARTREV C -> (none); STANDARD Manufacturer Recommendations -> (none)
- U3: MANUFACTURER Dialog Semicondutor -> (none); MAXIMUM_PACKAGE_HEIGHT 2.16mm -> (none); PARTREV F -> (none); STANDARD IPC 7351B -> (none)
Changed lines of the file:
@@
 F 2 "SOIC127P790X216-8N" H 2375 2225 50  0001 L BNN
 F 3 "https://www.dialog-semiconductor.com/sites/default/files/at25sf041b.pdf" H 2375 2225 50  0001 L BNN
-F 4 "IPC 7351B" H 2375 2225 50  0001 L BNN "STANDARD"
-F 5 "F" H 2375 2225 50  0001 L BNN "PARTREV"
-F 6 "Dialog Semicondutor" H 2375 2225 50  0001 L BNN "MANUFACTURER"
-F 7 "2.16mm" H 2375 2225 50  0001 L BNN "MAXIMUM_PACKAGE_HEIGHT"
-F 8 "IC FLASH 4MBIT SPI/QUAD 8SOIC" H 2375 2225 50  0001 C CNN "Desc"
-F 9 "1265-AT25SF041B-SHD-B-ND" H 2375 2225 50  0001 C CNN "PN_DIGIKEY"
-F 10 "0.36" H 2375 2225 50  0001 C CNN "PRICE_DIGIKEY"
+F 4 "IC FLASH 4MBIT SPI/QUAD 8SOIC" H 2375 2225 50  0001 C CNN "Desc"
+F 5 "1265-AT25SF041B-SHD-B-ND" H 2375 2225 50  0001 C CNN "PN_DIGIKEY"
+F 6 "0.36" H 2375 2225 50  0001 C CNN "PRICE_DIGIKEY"
 	1    2375 2225
 	1    0    0    -1
@@
 F 4 "CAP CER 1UF 10% 10V X7R 0805" H 3825 2150 50  0001 C CNN "Desc"
 F 5 "1uF" H 3250 2300 50  0000 C CNN "Comment"
-F 6 "399-1284-2-ND" H 3150 2225 50  0001 C CNN "PN_DIGIKEY"
+F 6 "399-1284-1-ND" H 3150 2225 50  0001 C CNN "PN_DIGIKEY"
 F 7 "0.14" H 3150 2225 50  0001 C CNN "PRICE_DIGIKEY"
 	1    3150 2225
@@
 F 4 "FERRITE BEAD 600 OHM 300mA 0805" V 5525 1975 50  0001 C CNN "Desc"
 F 5 "600R/0.3A" V 5375 1975 50  0000 C CNN "Comment"
-F 6 "490-11047-2-ND" H 5525 1975 50  0001 C CNN "PN_DIGIKEY"
+F 6 "490-11047-1-ND" H 5525 1975 50  0001 C CNN "PN_DIGIKEY"
 F 7 "0.18" H 5525 1975 50  0001 C CNN "PRICE_DIGIKEY"
 	1    5525 1975
@@
 	1    0    0    -1
 $EndComp
-$Comp
-L TC2030-IDC-NL:TC2030-IDC-NL J3
-U 1 1 615308AA
-P 4525 2175
-F 0 "J3" H 4468 2742 50  0000 C CNN
-F 1 "TC2030-IDC-NL" H 4468 2651 50  0000 C CNN
-F 2 "TAG_TC2030-IDC-NL" H 4525 2175 50  0001 L BNN
-F 3 "https://media.digikey.com/pdf/Data%20Sheets/Tag-Connect/TC2030-IDC_RevB.pdf" H 4525 2175 50  0001 L BNN
-F 4 "MS" H 4525 2175 50  0001 L BNN "PARTREV"
-F 5 "Tag-Connect" H 4525 2175 50  0001 L BNN "MANUFACTURER"
-F 6 "Manufacturer recommendation" H 4525 2175 50  0001 L BNN "STANDARD"
-F 7 "CABLE ADAPTER 6 POS" H 4525 2175 50  0001 C CNN "Desc"
-	1    4525 2175
-	-1   0    0    -1
-$EndComp
 Wire Wire Line
 	4825 1875 4900 1875
@@
 CSN
 $Comp
-L 1734592-8:1734592-8 J4
-U 1 1 615308E8
-P 4600 3875
-F 0 "J4" H 4800 3150 50  0000 L CNN
-F 1 "1734592-8" H 4450 3225 50  0000 L CNN
-F 2 "TE_1734592-8" H 4600 3875 50  0001 L BNN
-F 3 "https://www.te.com/commerce/DocumentDelivery/DDEController?Action=srchrtrv&DocNm=1734592&DocType=Customer+Drawing&DocLang=English" H 4600 3875 50  0001 L BNN
-F 4 "Manufacturer Recommendations" H 4600 3875 50  0001 L BNN "STANDARD"
-F 5 "TE Connectivity" H 4600 3875 50  0001 L BNN "MANUFACTURER"
-F 6 "2.05mm" H 4600 3875 50  0001 L BNN "MAXIMUM_PACKAGE_HEIGHT"
-F 7 "C" H 4600 3875 50  0001 L BNN "PARTREV"
-F 8 "CONN FPC BOTTOM 8POS 0.50MM R/A" H 4600 3875 50  0001 C CNN "Desc"
-F 9 "A100281TR-ND" H 4600 3875 50  0001 C CNN "PN_DIGIKEY"
-F 10 "0.46" H 4600 3875 50  0001 C CNN "PRICE_DIGIKEY"
-	1    4600 3875
-	-1   0    0    1
-$EndComp
-$Comp
 L power:GND #PWR018
 U 1 1 615308EE
@@
 Wire Wire Line
 	6800 1600 6800 1775
+$Comp
+L 1734592-8:1734592-8 J4
+U 1 1 615308E8
+P 4600 3875
+F 0 "J4" H 4800 3150 50  0000 L CNN
+F 1 "1734592-8" H 4450 3225 50  0000 L CNN
+F 2 "TE_1734592-8" H 4600 3875 50  0001 L BNN
+F 3 "https://www.te.com/commerce/DocumentDelivery/DDEController?Action=srchrtrv&DocNm=1734592&DocType=Customer+Drawing&DocLang=English" H 4600 3875 50  0001 L BNN
+F 4 "CONN FPC BOTTOM 8POS 0.50MM R/A" H 4600 3875 50  0001 C CNN "Desc"
+F 5 "A100281TR-ND" H 4600 3875 50  0001 C CNN "PN_DIGIKEY"
+F 6 "0.46" H 4600 3875 50  0001 C CNN "PRICE_DIGIKEY"
+	1    4600 3875
+	-1   0    0    1
+$EndComp
+$Comp
+L TC2030-IDC-NL:TC2030-IDC-NL J3
+U 1 1 615308AA
+P 4525 2175
+F 0 "J3" H 4468 2742 50  0000 C CNN
+F 1 "TC2030-IDC-NL" H 4468 2651 50  0000 C CNN
+F 2 "TAG_TC2030-IDC-NL" H 4525 2175 50  0001 L BNN
+F 3 "https://media.digikey.com/pdf/Data%20Sheets/Tag-Connect/TC2030-IDC_RevB.pdf" H 4525 2175 50  0001 L BNN
+F 4 "CABLE ADAPTER 6 POS" H 4525 2175 50  0001 C CNN "Desc"
+	1    4525 2175
+	-1   0    0    -1
+$EndComp
 $EndSCHEMATC
